File: eagle/Control board/control_board.sch (EAGLE design)
At the start: 237 parts, among them Q1 RE1C002UN, Q2 RE1C002UN, SW1 SPST_TACT-EVQQ2, SW2 SPST_TACT-EVQQ2, U1 TCA9554A, U2 LM317, U3 LM317, U4 STM32F446, U5 TCA9554A, U6 TCA9554A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

Commit message: Almost done routing
Parts:
- removed SB74, SB79, SB84, SB85, SB86, SB87, SB88, SB89, SB90, SB91, SB92, SB93, SB95, SB97: SOLDER_BRIDGE, custom:SOLDER_BRIDGE
- removed U3: LM317, custom:LM317TS
- added C10, C11: 22uF, rcl:C-EUC0603
- added U7: AZ1085CD, custom:AZ1085C
- C1, C2: value 0.1uF -> 10uF
- R1: value (none) -> 178
- R17, R8: value 82 -> 430
- R2: value (none) -> 287
- R3: value (none) -> 100
- R4: value (none) -> 301
- R7: value 430 -> 82
- U2: value LM317 -> AZ1085CD; device custom:LM317TS -> custom:AZ1085C
Connections:
- net PP8V_CONN renamed PP7V_CONN
- removed net MOTOR1_1EN: SB85.P$2, X9-4.S
- removed net MOTOR1_2EN: SB86.P$2, X9-5.S
- removed net MOTOR1_3EN: SB87.P$2, X9-6.S
- removed net MOTOR1_4EN: SB88.P$2, X9-7.S
- removed net MOTOR2_1EN: SB74.P$2, X10-4.S
- removed net MOTOR2_2EN: SB79.P$2, X10-5.S
- removed net MOTOR2_3EN: SB84.P$2, X10-6.S
- removed net MOTOR2_4EN: SB89.P$2, X10-7.S
- removed net MOTOR3_1EN: SB90.P$2, X11-4.S
- removed net MOTOR3_2EN: SB91.P$2, X11-5.S
- removed net MOTOR3_3EN: SB92.P$2, X11-6.S
- removed net MOTOR3_4EN: SB93.P$2, X11-7.S
- removed net SERVO1_PWM: SB95.P$2, X13-2.S
- removed net SERVO2_PWM: SB97.P$2, X14-2.S
- net GND: now also C10.2, C11.2
- net I2C2_SCL: now also SB120.P$1, SB70.P$1, SB75.P$1, SB80.P$1; no longer SB55.P$1, SB60.P$1, SB65.P$1
- net I2C2_SDA: now also SB119.P$1, SB71.P$1, SB76.P$1, SB81.P$1; no longer SB56.P$1, SB61.P$1, SB66.P$1
- net I2C3_SCL: now also SB55.P$1, SB60.P$1, SB65.P$1; no longer SB120.P$1, SB70.P$1, SB75.P$1, SB80.P$1
- net I2C3_SDA: now also SB56.P$1, SB61.P$1, SB66.P$1; no longer SB119.P$1, SB71.P$1, SB76.P$1, SB81.P$1
- net LED_3V3: now also LED1.A, R7.2; no longer LED2.A, R8.2
- net LED_5V: now also LED2.A, R8.2; no longer LED1.A, R7.2
- net M1_1: now also X9-4.S; no longer SB85.P$1
- net M1_2: now also X9-5.S; no longer SB86.P$1
- net M1_3: now also X9-6.S; no longer SB87.P$1
- net M1_4: now also X9-7.S; no longer SB88.P$1
- net M2_1: now also X10-4.S; no longer SB74.P$1
- net M2_2: now also X10-5.S; no longer SB79.P$1
- net M2_3: now also X10-6.S; no longer SB84.P$1
- net M2_4: now also X10-7.S; no longer SB89.P$1
- net M3_1: now also X11-4.S; no longer SB90.P$1
- net M3_2: now also X11-5.S; no longer SB91.P$1
- net M3_3: now also X11-6.S; no longer SB92.P$1
- net M3_4: now also X11-7.S; no longer SB93.P$1
- net N$1: now also U2.ADJ; no longer U3.ADJ
- net N$3: now also U7.ADJ; no longer U2.ADJ
- net PP3V3: now also C10.1, R1.1, R7.1, U7.OUT; no longer R17.1, R3.1, R8.1, U3.OUT
- net PP5V: now also C11.1, R17.1, R3.1, R8.1; no longer R1.1, R7.1
- net PP7V: now also U7.IN; no longer U3.IN
- net SERVO1: now also X13-2.S; no longer SB95.P$1
- net SERVO2: now also X14-2.S; no longer SB97.P$1
- net SW2: now also SB47.P$2; no longer SB49.P$2
- net SW3: now also SB49.P$2; no longer SB46.P$2
- net SW4: now also SB46.P$2; no longer SB47.P$2
Other:
- note added: "RF Initial I2C2 RF4 RF5 RF6 IMU_GYRO IMU_ACCEL IMU_MAG GPIO_EXPANDER3 I2C3 RF1 RF2 RF3 GPIO_EXPANDER1 GPIO_EXPANDER2"
- note removed: "RF Initial I2C2 RF1 RF2 RF3 IMU_GYRO IMU_ACCEL IMU_MAG I2C3 RF4 RF5 RF6 GPIO_EXPANDER1 GPIO_EXPANDER2 GPIO_EXPANDER3"
- moved on the sheet: C1, C2, LED1, LED2, R7, R8, X10-1, X10-2, X10-3, X10-4, X10-5, X10-6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

Commit message: Routing complete. Need GND stitching
Parts:
- removed SB53: SOLDER_BRIDGE, custom:SOLDER_BRIDGE
Connections:
- removed net PP7V_CONN: SB53.P$2, U4.VIN
- net PP7V: now also U4.VIN; no longer SB53.P$1
Changed lines of the file:
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@@
 <part name="SB49" library="custom" deviceset="SOLDER_BRIDGE" device=""/>
 <part name="SB50" library="custom" deviceset="SOLDER_BRIDGE" device=""/>
-<part name="SB53" library="custom" deviceset="SOLDER_BRIDGE" device=""/>
 <part name="R1" library="rcl" deviceset="R-US_" device="R0603" value="178"/>
 <part name="R2" library="rcl" deviceset="R-US_" device="R0603" value="287"/>
@@
 <instance part="SB49" gate="G$1" x="157.48" y="210.82"/>
 <instance part="SB50" gate="G$1" x="157.48" y="215.9"/>
-<instance part="SB53" gate="G$1" x="53.34" y="243.84"/>
 <instance part="SB51" gate="G$1" x="154.94" y="220.98" rot="MR0"/>
 <instance part="SB52" gate="G$1" x="154.94" y="226.06" rot="MR0"/>
@@
 </segment>
 </net>
-<net name="PP7V_CONN" class="0">
-<segment>
+<net name="PP7V" class="0">
+<segment>
+<label x="68.58" y="243.84" size="1.778" layer="95"/>
 <pinref part="U4" gate="G$1" pin="VIN"/>
 <wire x1="78.74" y1="233.68" x2="78.74" y2="243.84" width="0.1524" layer="91"/>
-<label x="60.96" y="243.84" size="1.778" layer="95"/>
-<wire x1="78.74" y1="243.84" x2="55.88" y2="243.84" width="0.1524" layer="91"/>
-<pinref part="SB53" gate="G$1" pin="P$2"/>
-</segment>
-</net>
-<net name="PP7V" class="0">
-<segment>
-<pinref part="SB53" gate="G$1" pin="P$1"/>
-<wire x1="48.26" y1="243.84" x2="33.02" y2="243.84" width="0.1524" layer="91"/>
-<label x="33.02" y="243.84" size="1.778" layer="95"/>
-</segment>
-</net>
+<wire x1="68.58" y1="243.84" x2="78.74" y2="243.84" width="0.1524" layer="91"/>
+</segment>
+</net>
