File: eagle/Control board/control_board.brd (EAGLE design)
At the start: 100 x 100 mm, 185 parts, among them Q1 RE1C002UN, Q2 RE1C002UN, SW1 SPST_TACT-EVQQ2, SW2 SPST_TACT-EVQQ2, U1 TCA9554A, U2 AZ1085CD, U4 STM32F446, U5 TCA9554A, U6 TCA9554A, U7 AZ1085CD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

Commit message: Routing complete. Need GND stitching
Parts:
- removed SB53: SOLDER_BRIDGE, custom:SOLDER_BRIDGE
- moved SW1 58.2 mm to (4.70, 11.8)
- moved SW2 40.7 mm to (16.0, 11.8)
- moved Q2 8.90 mm to (7.75, 73.5), turned to 0 degrees
- moved LED6 5.92 mm to (8.26, 77.1), turned to 180 degrees
- moved C1 3.51 mm to (90.9, 94.9), turned to 0 degrees
- moved R18 3.12 mm to (10.3, 77.1), turned to 90 degrees
- moved R21 2.11 mm to (35.8, 81.2), turned to 180 degrees
- moved LED5 2.03 mm to (86.9, 38.9)
- moved Q1 2.03 mm to (85.3, 41.7)
- moved R12 2.03 mm to (65.2, 83.1)
- moved R16 2.03 mm to (65.2, 90.4)
- moved R2 2.03 mm to (89.2, 87.1)
- moved R4 2.03 mm to (89.2, 76.2)
- moved SB12 2.03 mm to (79.9, 54.4)
- moved SB13 2.03 mm to (79.9, 56.9)
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Connections:
- removed net PP7V_CONN: SB53.P$2, U4.P$24
- net PP7V: now also U4.P$24; no longer SB53.P$1
Routing:
- net PP3V3: track 141.9 -> 305.0 mm, vias 4 -> 10
- net PP7V: track 36.7 -> 173.3 mm
- net RESET_BTN: track 6.80 -> 65.1 mm, vias 0 -> 1
- net DBG_BUTTON: track 6.80 -> 47.2 mm, vias 0 -> 1
- net LED_DBG2: track 9.88 -> 4.09 mm
- net PP7V_CONN: track 3.05 -> 0.00 mm
- net I2C2_SCL: track 80.8 -> 83.1 mm
- net PP12V: track 52.4 -> 53.6 mm
- net I2C3_SDA: track 107.9 -> 108.1 mm, vias 4 -> 5
- net I2C3_SCL: track 110.4 -> 110.5 mm, vias 4 -> 5
- added copper zone on layer 1, net GND
- added copper zone on layer 16, net GND

Commit message: GND stitching done
Routing:
- net PPBATT: track 56.7 -> 113.3 mm
- net PP12V: track 53.6 -> 72.1 mm
